Commit message: add

File: install/transport_robots/share/transport_robots/urdf/transport_robot.urdf.xacro (robot description, xacro)
@@ -71,4 +71,32 @@
   <xacro:wheel prefix="rear_left" x="${-wheel_offset_x}" y="${wheel_offset_y}"/>
   <xacro:wheel prefix="rear_right" x="${-wheel_offset_x}" y="${-wheel_offset_y}"/>
+  <!-- LiDAR sensor -->
+  <link name="lidar_link">
+    <visual>
+      <origin xyz="0 0 0" rpy="0 0 0"/>
+      <geometry>
+        <cylinder radius="0.05" length="0.04"/>
+      </geometry>
+      <material name="red">
+        <color rgba="0.8 0.2 0.2 1.0"/>
+      </material>
+    </visual>
+    <collision>
+      <origin xyz="0 0 0" rpy="0 0 0"/>
+      <geometry>
+        <cylinder radius="0.05" length="0.04"/>
+      </geometry>
+    </collision>
+    <inertial>
+      <origin xyz="0 0 0" rpy="0 0 0"/>
+      <mass value="0.1"/>
+      <inertia ixx="0.001" ixy="0.0" ixz="0.0" iyy="0.001" iyz="0.0" izz="0.001"/>
+    </inertial>
+  </link>
+  <joint name="lidar_joint" type="fixed">
+    <parent link="base_link"/>
+    <child link="lidar_link"/>
+    <origin xyz="0 0 ${base_height/2 + 0.02}" rpy="0 0 0"/>
+  </joint>
   <!-- Gazebo plugins -->
   <gazebo>
@@ -93,4 +121,40 @@
     </plugin>
   </gazebo>
+  <!-- LiDAR Gazebo plugin -->
+  <gazebo reference="lidar_link">
+    <sensor type="ray" name="lidar_sensor">
+      <pose>0 0 0 0 0 0</pose>
+      <visualize>true</visualize>
+      <update_rate>10</update_rate>
+      <ray>
+        <scan>
+          <horizontal>
+            <samples>360</samples>
+            <resolution>1</resolution>
+            <min_angle>-3.14159</min_angle>
+            <max_angle>3.14159</max_angle>
+          </horizontal>
+        </scan>
+        <range>
+          <min>0.1</min>
+          <max>10.0</max>
+          <resolution>0.01</resolution>
+        </range>
+        <noise>
+          <type>gaussian</type>
+          <mean>0.0</mean>
+          <stddev>0.01</stddev>
+        </noise>
+      </ray>
+      <plugin name="gazebo_ros_lidar_controller" filename="libgazebo_ros_ray_sensor.so">
+        <ros>
+          <namespace>$(arg robot_name)</namespace>
+          <remapping>~/out:=scan</remapping>
+        </ros>
+        <output_type>sensor_msgs/LaserScan</output_type>
+        <frame_name>lidar_link</frame_name>
+      </plugin>
+    </sensor>
+  </gazebo>
   <!-- Gazebo materials -->
   <gazebo reference="base_link">

Commit message: add

File: install/transport_robots/share/transport_robots/urdf/transport_robot.urdf.xacro (robot description, xacro)
@@ -30,7 +30,14 @@
     </collision>
     <inertial>
-      <origin xyz="0 0 0" rpy="0 0 0"/>
+      <origin xyz="-0.3 0 0" rpy="0 0 0"/>
       <mass value="20.0"/>
-      <inertia ixx="1.0" ixy="0.0" ixz="0.0" iyy="1.0" iyz="0.0" izz="1.0"/>
+      <!-- 正確な慣性テンソルを計算 -->
+      <inertia
+        ixx="${(1.0/12.0) * 20.0 * (base_width*base_width + base_height*base_height)}"
+        ixy="0.0"
+        ixz="0.0"
+        iyy="${(1.0/12.0) * 20.0 * (base_length*base_length + base_height*base_height)}"
+        iyz="0.0"
+        izz="${(1.0/12.0) * 20.0 * (base_length*base_length + base_width*base_width)}"/>
     </inertial>
   </link>
@@ -56,5 +63,12 @@
         <origin xyz="0 0 0" rpy="1.5708 0 0"/>
         <mass value="2.0"/>
-        <inertia ixx="0.1" ixy="0.0" ixz="0.0" iyy="0.1" iyz="0.0" izz="0.1"/>
+        <!-- 円柱の慣性テンソル -->
+        <inertia
+          ixx="${(1.0/12.0) * 2.0 * (3*wheel_radius*wheel_radius + wheel_width*wheel_width)}"
+          ixy="0.0"
+          ixz="0.0"
+          iyy="${(1.0/12.0) * 2.0 * (3*wheel_radius*wheel_radius + wheel_width*wheel_width)}"
+          iyz="0.0"
+          izz="${0.5 * 2.0 * wheel_radius*wheel_radius}"/>
       </inertial>
     </link>
@@ -106,6 +120,6 @@
       </ros>
       <update_rate>30</update_rate>
-      <left_joint>front_left_wheel_joint</left_joint>
-      <right_joint>front_right_wheel_joint</right_joint>
+      <left_joint>rear_left_wheel_joint</left_joint>
+      <right_joint>rear_right_wheel_joint</right_joint>
       <wheel_separation>${base_width}</wheel_separation>
       <wheel_diameter>${2*wheel_radius}</wheel_diameter>
@@ -119,4 +133,9 @@
       <odometry_frame>odom</odometry_frame>
       <robot_base_frame>base_link</robot_base_frame>
+      <!-- 重要: 回転中心を後輪軸に設定 -->
+      <wheel_separation>${base_width}</wheel_separation>
+      <wheel_diameter>${2*wheel_radius}</wheel_diameter>
+      <!-- オドメトリの基準点を調整 -->
+      <odometry_source>world</odometry_source>
     </plugin>
   </gazebo>
